File: 48_buck.brd (EAGLE design)
At the start: 100 x 80 mm, 31 parts

Commit message: Update with values from quickstart sheet
Parts:
- removed R13: 10K, rcl:RTRIM3224W
- added C16: 1uF, rcl:C1206
- added C17: .1uF, rcl:C0805
- added C18: .01uF, rcl:C0805
- added D1, D2: (no value), zetex:SOT-23
- added J1, J2: POWERPOLE_POWER45A_HORIZONTAL_DRILL, powerpoles:POWERPOLE_PAIR_45A_HORIZ_HOLE
- added J3: POWERPOLE_POWER10AWG, powerpoles:POWERPOLE_PAIR_10AWG
- added Q1, Q2: BUZ21, transistor-fet:TO220
- C1: value 220uF -> 61.2uF; device rcl:EB25D -> rcl:C0805
- C10, C11, C12, C13: value 100uF -> 330uF; device rcl:C0805 -> resistor:E5-10,5
- C14: device rcl:C0805 -> rcl:C1210
- C15: value 100uF -> 10uF; device rcl:C0805 -> rcl:C1206
- C3: value .22uF -> 910pF
- C4: value 560pF -> 33pF
- C5: value (none) -> 0.1uF
- C6: value (none) -> 1100pF
- C7: value 100uF -> 1uF
- C8: value 1uF -> 0.47uF
- C9: value 100uF -> 1uF; device rcl:C0805 -> rcl:C1206
- L1: value 15uH -> 10uH; device rcl:0207/15 -> rcl:TJ5-U2
- R1: value 390K -> 75K; device rcl:R0805 -> rcl:R1206
- R10: value 1M -> 10K2
- R11: value 315K -> 1K; device rcl:R0805 -> rcl:RTRIM3224W
- R12: value 10K -> 3m 1%
- R2: value 11K -> 500R; device rcl:R0805 -> rcl:RTRIM3224W
- R3: value 12.4K -> 1K8; device rcl:R0805 -> rcl:R1206
- R4: value (none) -> 1M
- R5: value 1K -> 300K
- R6: value 1k -> 12.4K
- R7: value 3m -> 71K5
- R8: value 1M -> 634K
- R9: value 300K -> 1K
- moved R2 193.1 mm to (-17.8, -228.6)
- moved C2 175.3 mm to (-20.3, -241.3)
- moved R12 149.9 mm to (-20.3, -61.0)
- moved C7 130.5 mm to (-59.7, -284.5)
- moved C9 100.3 mm to (-20.3, -66.0)
- moved R5 91.4 mm to (-20.3, -142.2)
- moved R4 91.4 mm to (-20.3, -137.2)
- moved R9 86.4 mm to (-20.3, -55.9)
- moved C15 67.3 mm to (-59.7, -259.1)
- moved R11 66.1 mm to (-17.8, -219.7)
- moved R10 63.5 mm to (-20.3, -210.8)
- moved C14 38.1 mm to (-20.3, -160.0)
- moved R8 16.5 mm to (-20.3, -153.7)
- moved R6 15.2 mm to (-20.3, -40.6)
- moved R7 15.2 mm to (-20.3, -45.7)
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- renumbered U$1 to LM5116
Connections:
- removed net N$13: R12.1, R13.2, R5.2
- removed net V+: C1.+, LM5116.1, R1.2, R8.2
- new net N$16: R10.1, R11.2, R11.3
- new net N$17: C1.1, D2.1, J2.RED, J3.RED, LM5116.1, Q1.2, R1.2, R4.2
- new net N$19: C4.2, LM5116.8, R10.2, R7.2, R9.1
- new net N$20: C8.2, L1.1, LM5116.20, Q1.3, Q2.2
- net GND: now also C2.2, C5.2, C6.2, R3.1, R9.2; no longer C3.2, C4.2, LM5116.17, R2.2, R3.2
- net N$1: now also R2.2, R3.2; no longer LM5116.2, R1.1, R2.1
- net N$10: now also C8.1, D1.1, LM5116.18; no longer C8.2, L1.1, LM5116.20
- net N$11: now also C2.1, D2.3, LM5116.2, R1.1, R2.1; no longer C10.1, C11.1, C12.1, C13.1, C14.1, C15.1, C7.1, C9.1, L1.2, LM5116.10, R13.1, R5.1
- net N$12: now also LM5116.19, Q1.1; no longer C8.1, LM5116.18
- net N$14: now also C10.+, C11.+, C12.+, C13.+, C14.1, C15.1, C16.1, C17.1, C18.1, C7.1, J1.RED, L1.2, LM5116.10, LM5116.17, R11.1; no longer JP1.2, LM5116.4, R10.2
- net N$15: now also Q2.3, R12.1; no longer R7.1
- net N$2: now also LM5116.4, R4.1, R5.2; no longer R8.1, R9.2
- net N$3: now also C5.1; no longer C3.1
- net N$4: now also C9.1, D1.3, R8.2; no longer C2.1, R11.2
- net N$5: now also C3.2, R7.1; no longer C5.2, R4.1
- net N$6: now also R6.1; no longer R3.1
- net N$7: now also C3.1, C4.1; no longer C5.1, C6.1
- net N$8: now also LM5116.15, Q2.1; no longer C6.2, LM5116.8, R12.2, R4.2, R6.1
- net N$9: now also C6.1, R8.1; no longer C4.1, R11.1
- net PE: now also C1.2, C10.-, C11.-, C12.-, C13.-, C16.2, C17.2, C18.2, J1.BLACK, J2.BLACK, J3.BLACK, JP1.2, R12.2, R5.1; no longer C1.-, C10.2, C11.2, C12.2, C13.2, C2.2, R10.1, R7.2, R9.1

Commit message: Verified schematic, added components to library, started layout
Parts:
- added C19, C20: 22uF, rcl:E3,5-8
- C1: value 61.2uF -> 22uF; device rcl:C0805 -> rcl:E3,5-8
- C2: device rcl:C0805 -> rcl:C1206
- L1: device rcl:TJ5-U2 -> 48buck_library:AIRD-03
- R10: device rcl:R0805 -> 48buck_library:R2818
- R11: device rcl:RTRIM3224W -> 48buck_library:3303X-3
- R2: value 500R -> 500; device rcl:RTRIM3224W -> 48buck_library:3303X-3
- moved C7 375.3 mm to (-36.8, 90.2)
- moved D2 371.3 mm to (-47.0, 73.7)
- moved D1 366.2 mm to (-43.2, 73.7)
- moved C17 363.5 mm to (-26.7, 90.2)
- moved C18 362.1 mm to (-49.5, 83.8)
- moved C16 349.7 mm to (-77.5, 83.8)
- moved C15 342.9 mm to (-55.9, 83.8)
- moved C2 328.5 mm to (-67.3, 83.8)
- moved Q2 326.6 mm to (-30.5, 44.5)
- moved Q1 326.4 mm to (-19.1, 44.5)
- moved R2 318.8 mm to (-47.0, 88.9)
- moved J2 315.6 mm to (15.2, 74.9)
- moved R11 311.0 mm to (-55.9, 88.9)
- moved J3 280.9 mm to (12.2, 22.3)
- moved R10 277.1 mm to (-49.5, 64.8)
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Connections:
- net N$1: now also R2.1; no longer R2.2
- net N$11: now also R2.2; no longer R2.1
- net N$14: now also L1.P$2, R11.3; no longer L1.2, R11.1
- net N$16: now also R10.P$1, R11.1; no longer R10.1, R11.3
- net N$17: now also C1.+, C19.+, C20.+; no longer C1.1
- net N$19: now also R10.P$2; no longer R10.2
- net N$20: now also L1.P$1; no longer L1.1
- net PE: now also C1.-, C19.-, C20.-; no longer C1.2
